File: pcb-psu-led.kicad_pcb (KiCad board)
At the start: 2 copper layers, 142 x 50 mm, 20 parts, among them J1 Phoenix_MSTBA_2pin_P5.08, J2 JST_XH_B2B_2pin_P2.5, T1 Talema_70000K_1p6VA, U1 TO92_LM78L05

Commit message: pcb-psu-led.kicad_pcb
Routing:
- net ZERO_V_LED: track 0.00 -> 135.6 mm
- net VRAW_PLUS: track 0.00 -> 94.8 mm
- net L_SW: track 0.00 -> 63.5 mm
- net N_SW: track 0.00 -> 58.5 mm
- net LED_R1_OUT: track 0.00 -> 42.6 mm
- net PLUS_5V_LED: track 0.00 -> 35.7 mm
- net LED_DRIVE: track 0.00 -> 28.2 mm
- net PRI_LINK_5_4: track 0.00 -> 25.4 mm
- net SEC_B: track 0.00 -> 21.1 mm
- net SEC_A: track 0.00 -> 9.46 mm
Other:
- board text added: "CAUTION: 230 VAC PRIMARY"
Changed lines of the file:
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@@
     (title "PCB PSU LED — Stepdown 230/100 V")
     (date "2026-07-14")
-    (rev "PLACEMENT 0.1")
+    (rev "ROUTED CANDIDATE 1.0")
     (company "Piotr Koszalka")
     (comment 1 "Talema 70000K, isolated floating SELV output")
-    (comment 2 "142 x 50 mm — placement review, unrouted")
+    (comment 2 "142 x 50 mm — routed manufacturing candidate")
   )
   (layers
@@
 )
   )
+  (segment (start 7.46 25) (end 7.46 35) (width 1) (layer "F.Cu") (net 1))
+  (segment (start 7.46 35) (end 20 35) (width 1) (layer "F.Cu") (net 1))
+  (segment (start 20 35) (end 20 42.78) (width 1) (layer "F.Cu") (net 1))
+  (segment (start 20 42.78) (end 53.22 42.78) (width 1) (layer "F.Cu") (net 1))
+  (segment (start 12.54 25) (end 12.54 15) (width 1) (layer "F.Cu") (net 2))
+  (segment (start 12.54 15) (end 28 15) (width 1) (layer "F.Cu") (net 2))
+  (segment (start 28 15) (end 28 7.22) (width 1) (layer "F.Cu") (net 2))
+  (segment (start 28 7.22) (end 53.22 7.22) (width 1) (layer "F.Cu") (net 2))
+  (segment (start 53.22 12.3) (end 53.22 37.7) (width 1) (layer "B.Cu") (net 3))
+  (segment (start 88.78 7.22) (end 92 7.22) (width 1) (layer "F.Cu") (net 4))
+  (segment (start 92 7.22) (end 98 8.92) (width 1) (layer "F.Cu") (net 4))
+  (segment (start 88.78 42.78) (end 92 42.78) (width 1) (layer "F.Cu") (net 5))
+  (segment (start 92 42.78) (end 92 30.92) (width 1) (layer "F.Cu") (net 5))
+  (segment (start 92 30.92) (end 98 30.92) (width 1) (layer "F.Cu") (net 5))
+  (segment (start 98 19.08) (end 103 19.08) (width 0.8) (layer "F.Cu") (net 7))
+  (segment (start 103 19.08) (end 106.75 25) (width 0.8) (layer "F.Cu") (net 7))
+  (segment (start 98 41.08) (end 103 41.08) (width 0.8) (layer "F.Cu") (net 7))
+  (segment (start 103 41.08) (end 103 28.75) (width 0.8) (layer "F.Cu") (net 7))
+  (segment (start 103 28.75) (end 106.75 25) (width 0.8) (layer "F.Cu") (net 7))
+  (segment (start 106.75 25) (end 106.75 35) (width 0.8) (layer "F.Cu") (net 7))
+  (segment (start 106.75 25) (end 110 25) (width 0.8) (layer "F.Cu") (net 7))
+  (segment (start 110 25) (end 110 19) (width 0.8) (layer "F.Cu") (net 7))
+  (segment (start 110 19) (end 114 19) (width 0.8) (layer "F.Cu") (net 7))
+  (segment (start 114 19) (end 112 22) (width 0.8) (layer "F.Cu") (net 7))
+  (segment (start 112 22) (end 112 32) (width 0.8) (layer "F.Cu") (net 7))
+  (segment (start 112 32) (end 122.27 32) (width 0.8) (layer "F.Cu") (net 7))
+  (segment (start 122.27 32) (end 122.27 25) (width 0.8) (layer "F.Cu") (net 7))
+  (segment (start 110 19) (end 110 13) (width 0.8) (layer "F.Cu") (net 7))
+  (segment (start 88.78 12.3) (end 94 12.3) (width 0.8) (layer "B.Cu") (net 6))
+  (segment (start 94 12.3) (end 94 25) (width 0.8) (layer "B.Cu") (net 6))
+  (segment (start 94 25) (end 109.25 25) (width 0.8) (layer "B.Cu") (net 6))
+  (segment (start 88.78 37.7) (end 94 37.7) (width 0.8) (layer "B.Cu") (net 6))
+  (segment (start 94 37.7) (end 94 25) (width 0.8) (layer "B.Cu") (net 6))
+  (segment (start 109.25 25) (end 109.25 35) (width 0.8) (layer "B.Cu") (net 6))
+  (segment (start 108.75 35) (end 109.25 35) (width 0.8) (layer "B.Cu") (net 6))
+  (segment (start 109.25 25) (end 109.25 30) (width 0.8) (layer "B.Cu") (net 6))
+  (segment (start 109.25 30) (end 138.25 30) (width 0.8) (layer "B.Cu") (net 6))
+  (segment (start 138.25 30) (end 138.25 25) (width 0.8) (layer "B.Cu") (net 6))
+  (segment (start 119 19) (end 119 30) (width 0.5) (layer "B.Cu") (net 6))
+  (segment (start 121 25) (end 121 30) (width 0.5) (layer "B.Cu") (net 6))
+  (segment (start 128.5 19) (end 128.5 30) (width 0.5) (layer "B.Cu") (net 6))
+  (segment (start 118 38) (end 118 30) (width 0.5) (layer "B.Cu") (net 6))
+  (segment (start 119.73 25) (end 119.73 16) (width 0.5) (layer "F.Cu") (net 8))
+  (segment (start 119.73 16) (end 123.5 16) (width 0.5) (layer "F.Cu") (net 8))
+  (segment (start 123.5 16) (end 123.5 19) (width 0.5) (layer "F.Cu") (net 8))
+  (segment (start 119.73 16) (end 116 12) (width 0.5) (layer "F.Cu") (net 8))
+  (segment (start 116 12) (end 111 12) (width 0.5) (layer "F.Cu") (net 8))
+  (segment (start 111 12) (end 111 8) (width 0.5) (layer "F.Cu") (net 8))
+  (segment (start 123.5 16) (end 127 16) (width 0.5) (layer "F.Cu") (net 8))
+  (segment (start 127 16) (end 127 14) (width 0.5) (layer "F.Cu") (net 8))
+  (segment (start 126 8) (end 131 8) (width 0.5) (layer "F.Cu") (net 9))
+  (segment (start 131 8) (end 134 11) (width 0.5) (layer "F.Cu") (net 9))
+  (segment (start 134 11) (end 134 34) (width 0.5) (layer "F.Cu") (net 9))
+  (segment (start 134 34) (end 128 39) (width 0.5) (layer "F.Cu") (net 9))
+  (segment (start 128 39) (end 125.46 39) (width 0.5) (layer "F.Cu") (net 9))
+  (segment (start 130.54 39) (end 135.75 39) (width 0.5) (layer "F.Cu") (net 10))
+  (segment (start 135.75 39) (end 135.75 25) (width 0.5) (layer "F.Cu") (net 10))
+  (segment (start 135.75 25) (end 136 16) (width 0.5) (layer "F.Cu") (net 10))
   (gr_line (start 0 0) (end 142 0) (stroke (width 0.1) (type default)) (layer "Edge.Cuts"))
   (gr_line (start 142 0) (end 142 50) (stroke (width 0.1) (type default)) (layer "Edge.Cuts"))
@@
   (gr_line (start 75 1) (end 75 49) (stroke (width 0.25) (type dash)) (layer "Dwgs.User"))
   (dimension (type aligned) (layer "Dwgs.User") (pts (xy 0 0) (xy 142 0)) (height -5) (gr_text "142.00 mm" (at 71 -6.15 0) (layer "Dwgs.User") (effects (font (size 1.27 1.27) (thickness 0.15)))) (format (units 3) (units_format 1) (precision 2)))
-  (dimension (type aligned) (layer "Dwgs.User") (pts (xy 142 0) (xy 142 50)) (height -5) (gr_text "50.00 mm" (at 148.15 25 90) (layer "Dwgs.User") (effects (font (size 1.27 1.27) (thickness 0.15)))) (format (units 3) (units_format 1) (precision 2)))
-)
+  (dimension (type aligned) (layer "Dwgs.User") (pts (xy 142 0) (xy 142 50)) (height -5) (gr_text "50.00 mm" (at 148.15 25 90) (layer "Dwgs.User") (effects (font (size 1.27 1.27) (thickness 0.15)))) (format (units 3) (units_format 1) (precision 2)))  (gr_text "CAUTION: 230 VAC PRIMARY" (at 31 47 0) (layer "B.SilkS")
+    (effects (font (size 1 1) (thickness 0.15)) (justify mirror)))
+)
